File: board/PS2toADB/PS2toADB.kicad_sch (KiCad schematic)
At the start: 7 parts, among them U1 PIC12F1840

Commit message: Updated schematic. Added power button and renders
Parts:
- removed D1: 1N4148, Diode_THT:D_DO-35_SOD27_P2.54mm_Vertical_KathodeUp, symbol Diode:1N4148
- added C1: 10 uF, Capacitor_THT:CP_Radial_D5.0mm_P2.00mm, symbol Device:C_Polarized
- added C3, C4: 470 nF, Capacitor_THT:C_Disc_D3.0mm_W1.6mm_P2.50mm, symbol Device:C
- added R1, R2: 5K, Resistor_THT:R_Axial_DIN0204_L3.6mm_D1.6mm_P2.54mm_Vertical, symbol Device:R
- added R4: 10K, Resistor_THT:R_Axial_DIN0204_L3.6mm_D1.6mm_P2.54mm_Vertical, symbol Device:R
- added SW1: PowerOn, Button_Switch_THT:SW_PUSH_6mm_H5mm, symbol Switch:SW_Push
- J1: renamed from ADB_J1; value Mini-DIN-4 -> ADB
- J2: renamed from PS2KBD_J2; value Mini-DIN-6 -> PS/2 Keyboard
- J3: renamed from PS2MSE_J3; value Mini-DIN-6 -> PS/2 Mouse
- R3: renamed from R1; value 100 -> 5K
- renumbered C1 to C2
Connections:
- net PS2_KBD_DATA is gone; now on net PS2_DTK: J2.1
- net ADB_DATA: now also R4.2
- net GND: now also C1.2, C3.2, C4.2
- net PS2_CLK: now also R1.2
- net VCC: now also J2.4, J3.4, C1.1, C3.1, C4.1, R1.1, R2.1, R4.1, SW1.1
- net PS2_DTK: now reaches U1.4 (RA3)
- net PS2_DTK: now also R2.2
- net ADB_PWRON: now reaches J1.2
- net ADB_PWRON: now also SW1.2
- net PS2_MSE_DATA renamed PS2_DTM
- no-connect marks 9 -> 6
Other:
- moved on the sheet: C2, J2, J3, R3
